Commit message: added the rest of the modifications

File: robot_model_and_simulation/urdf/robot.xacro (robot description, xacro)
@@ -29,296 +29,3 @@
     <!-- Control Parameters -->
     <xacro:property name="max_linear_acceleration" value="10"/>
-    <!-- Links -->
-    <!-- Body Link -->
-    <link name="body_link">
-        <visual>
-            <origin xyz="0.0 0.0 0.0" rpy="0.0 0.0 0.0"/>
-            <geometry>
-                <box size="${body_length} ${body_width} ${body_height}"/>
-            </geometry>
-            <material name="body_material">
-                <color rgba="0.25 0.25 0.25 1.0"/>
-            </material>
-        </visual>
-        <collision>
-            <origin xyz="0.0 0.0 0.0" rpy="0.0 0.0 0.0"/>
-            <geometry>
-                <box size="${body_length} ${body_width} ${body_height}"/>
-            </geometry>
-        </collision>
-        <inertial>
-            <mass value="10"/>
-            <inertia ixx="${body_inertia_x}" ixy="0.0" ixz="0.0" iyy="${body_inertia_y}" iyz="0" izz="${body_inertia_z}"/>
-            <origin xyz="0 0 0" rpy="0 0 0"/>
-        </inertial>
-    </link>
-    <!-- Left Wheel -->
-    <link name="left_wheel_link">
-        <visual>
-            <origin xyz="0.0 0.0 0.0" rpy="1.570795 0.0 0.0"/>
-            <geometry>
-                <cylinder radius="${wheel_radius}" length="${wheel_width}"/>
-            </geometry>
-            <material name="wheel_material">
-                <color rgba="0.0 0.0 0.0 1.0"/>
-            </material>
-        </visual>
-        <collision>
-            <origin xyz="0.0 0.0 0.0" rpy="1.570795 0.0 0.0"/>
-            <geometry>
-                <cylinder radius="${wheel_radius}" length="${wheel_width}"/>
-            </geometry>
-        </collision>
-        <inertial>
-            <mass value="2"/>
-            <inertia ixx="${wheel_inertia_x}" ixy="0.0" ixz="0.0" iyy="${wheel_inertia_y}" iyz="0" izz="${wheel_inertia_z}"/>
-            <origin xyz="0.0 0.0 0.0" rpy="1.570795 0.0 0.0"/>
-        </inertial>
-    </link>
-    <!-- Right Wheel -->
-    <link name="right_wheel_link">
-        <visual>
-            <origin xyz="0.0 0.0 0.0" rpy="1.570795 0.0 0.0"/>
-            <geometry>
-                <cylinder radius="${wheel_radius}" length="${wheel_width}"/>
-            </geometry>
-            <material name="wheel_material">
-                <color rgba="0.0 0.0 0.0 1.0"/>
-            </material>
-        </visual>
-        <collision>
-            <origin xyz="0.0 0.0 0.0" rpy="1.570795 0.0 0.0"/>
-            <geometry>
-                <cylinder radius="${wheel_radius}" length="${wheel_width}"/>
-            </geometry>
-        </collision>
-        <inertial>
-            <mass value="2"/>
-            <inertia ixx="${wheel_inertia_x}" ixy="0.0" ixz="0.0" iyy="${wheel_inertia_y}" iyz="0" izz="${wheel_inertia_z}"/>
-            <origin xyz="0.0 0.0 0.0" rpy="1.570795 0.0 0.0"/>
-        </inertial>
-    </link>
-    <!-- Caster Wheel -->
-    <link name="caster_link">
-        <visual>
-            <origin xyz="0.0 0.0 0.0" rpy="0.0 0.0 0.0"/>
-            <geometry>
-                <sphere radius="${caster_radius}"/>
-            </geometry>
-            <material name="caster_material">
-                <color rgba="0.0 0.0 0.0 1.0"/>
-            </material>
-        </visual>
-        <collision>
-            <origin xyz="0.0 0.0 0.0" rpy="0.0 0.0 0.0"/>
-            <geometry>
-                <sphere radius="${caster_radius}"/>
-            </geometry>
-        </collision>
-        <inertial>
-            <mass value="0.5"/>
-            <inertia ixx="${caster_inertia_x}" ixy="0.0" ixz="0.0" iyy="${caster_inertia_y}" iyz="0" izz="${caster_inertia_z}"/>
-            <origin xyz="0 0 0" rpy="0 0 0"/>
-        </inertial>
-    </link>
-    <!-- Joints -->
-    <!-- Left Wheel Joint -->
-    <joint name="left_wheel_joint" type="continuous">
-        <origin xyz="-${wheel_offset} ${wheel_separation/2} -${wheel_radius/2}" rpy="0 0 0"/>
-        <parent link="body_link"/>
-        <child link="left_wheel_link"/>
-        <axis xyz="0 1 0"/>
-        <limit effort="100" velocity="10.0"/>
-        <dynamics damping="0.1" friction="0.1"/>
-    </joint>
-    <!-- Right Wheel Joint -->
-    <joint name="right_wheel_joint" type="continuous">
-        <origin xyz="-${wheel_offset} ${-wheel_separation/2} -${wheel_radius/2}" rpy="0 0 0"/>
-        <parent link="body_link"/>
-        <child link="right_wheel_link"/>
-        <axis xyz="0 1 0"/>
-        <limit effort="100" velocity="10.0"/>
-        <dynamics damping="0.1" friction="0.1"/>
-    </joint>
-    <!-- Caster Wheel Joint (fixed) -->
-    <joint name="caster_joint" type="fixed">
-        <origin xyz="${caster_offset} 0 -${caster_radius/2}" rpy="0 0 0"/>
-        <parent link="body_link"/>
-        <child link="caster_link"/>
-    </joint>
-      <!-- camera -->
-  <joint type="fixed" name="camera_joint">
-    <origin xyz="0.240 0 0.135" rpy="0 0 0"/>
-    <child link="camera_link"/>
-    <parent link="body_link"/>
-    <axis xyz="0 1 0" />
-  </joint>
-  <link name='camera_link'>
-    <pose>0 0 0 0 0 0</pose>
-    <inertial>
-      <mass value="0.1"/>
-      <origin xyz="0 0 0" rpy="0 0 0"/>
-      <inertia
-          ixx="1e-6" ixy="0" ixz="0"
-          iyy="1e-6" iyz="0"
-          izz="1e-6"
-      />
-    </inertial>
-    <collision name='collision'>
-      <origin xyz="0 0 0" rpy="0 0 0"/>
-      <geometry>
-        <box size=".03 .03 .03"/>
-      </geometry>
-    </collision>
-    <visual name='camera_link_visual'>
-      <origin xyz="0 0 0" rpy="0 0 0"/>
-      <geometry>
-        <box size=".03 .03 .03"/>
-      </geometry>
-    </visual>
-  </link>
-  <gazebo reference="camera_link">
-    <material>Gazebo/Red</material>
-  </gazebo>
-  <joint type="fixed" name="camera_optical_joint">
-    <origin xyz="0 0 0" rpy="-1.5707 0 -1.5707"/>
-    <child link="camera_link_optical"/>
-    <parent link="camera_link"/>
-  </joint>
-  <link name="camera_link_optical">
-  </link>
-   <!-- - Lidar -->
-  <joint type="fixed" name="scan_joint">
-     <origin xyz="0.250 0 0.075" rpy="0 0 0"/>
-    <child link="scan_link"/>
-    <parent link="body_link"/>
-    <axis xyz="0 1 0" rpy="0 0 0"/>
-  </joint>
-  <link name='scan_link'>
-    <inertial>
-      <mass value="1e-5"/>
-      <origin xyz="0 0 0" rpy="0 0 0"/>
-      <inertia
-          ixx="1e-6" ixy="0" ixz="0"
-          iyy="1e-6" iyz="0"
-          izz="1e-6"
-      />
-    </inertial>
-    <collision name='collision'>
-      <origin xyz="0 0 0" rpy="0 0 0"/>
-      <geometry>
-        <box size=".1 .1 .1"/>
-      </geometry>
-    </collision>
-    <visual name='scan_link_visual'>
-      <origin xyz="0 0 0" rpy="0 0 0"/>
-      <geometry>
-         <box size=".1 .1 .1"/>
-      </geometry>
-    </visual>
-  </link>
-    <!-- Gazebo Parameters -->
-    <gazebo reference="body_link">
-        <mu1>1.0</mu1>
-        <mu2>1.0</mu2>
-    </gazebo>
-    <gazebo reference="right_wheel_link">
-        <mu1>1.0</mu1>
-        <mu2>1.0</mu2>
-    </gazebo>
-    <gazebo reference="left_wheel_link">
-        <mu1>1.0</mu1>
-        <mu2>1.0</mu2>
-    </gazebo>
-    <gazebo reference="caster_link">
-        <mu1>0.000001</mu1>
-        <mu2>0.000001</mu2>
-    </gazebo>
-    <!-- Gazebo Plugins -->
-    <gazebo>
-        <plugin filename="gz-sim-diff-drive-system" name="gz::sim::systems::DiffDrive">
-            <right_joint>right_wheel_joint</right_joint>
-            <left_joint>left_wheel_joint</left_joint>
-            <wheel_separation>${wheel_separation}</wheel_separation>
-            <wheel_radius>${wheel_radius}</wheel_radius>
-            <max_linear_acceleration>${max_linear_acceleration}</max_linear_acceleration>
-            <odom_publish_frequency>100</odom_publish_frequency>
-            <topic>robot_vel</topic>
-            <odom_topic>odom</odom_topic>
-        </plugin>
-    </gazebo>
-<gazebo reference="camera_link">
-    <sensor name="camera" type="camera">
-      <camera>
-        <horizontal_fov>1.3962634</horizontal_fov>
-        <image>
-          <width>640</width>
-          <height>480</height>
-          <format>R8G8B8</format>
-        </image>
-        <clip>
-          <near>0.1</near>
-          <far>15</far>
-        </clip>
-        <noise>
-          <type>gaussian</type>
-          <!-- Noise is sampled independently per pixel on each frame.
-               That pixel's noise value is added to each of its color
-               channels, which at that point lie in the range [0,1]. -->
-          <mean>0.0</mean>
-          <stddev>0.007</stddev>
-        </noise>
-        <optical_frame_id>camera_link_optical</optical_frame_id>
-        <camera_info_topic>camera/camera_info</camera_info_topic>
-      </camera>
-      <always_on>1</always_on>
-      <update_rate>20</update_rate>
-      <visualize>true</visualize>
-      <topic>camera/image</topic>
-    </sensor>
-  </gazebo>
-  <gazebo reference="scan_link">
-    <sensor name="gpu_lidar" type="gpu_lidar">
-      <update_rate>10</update_rate>
-      <topic>scan</topic>
-      <gz_frame_id>scan_link</gz_frame_id>
-      <lidar>
-        <scan>
-          <horizontal>
-            <samples>720</samples>
-            <!--(max_angle-min_angle)/samples * resolution -->
-            <resolution>1</resolution>
-            <min_angle>-3.14156</min_angle>
-            <max_angle>3.14156</max_angle>
-          </horizontal>
-          <!-- Dirty hack for fake lidar detections with ogre 1 rendering in VM -->
-          <!-- <vertical>
-              <samples>3</samples>
-              <min_angle>-0.001</min_angle>
-              <max_angle>0.001</max_angle>
-          </vertical> -->
-        </scan>
-        <range>
-          <min>0.05</min>
-          <max>10.0</max>
-          <resolution>0.01</resolution>
-        </range>
-        <noise>
-            <type>gaussian</type>
-            <mean>0.0</mean>
-            <stddev>0.01</stddev>
-        </noise>
-        <frame_id>scan_link</frame_id>
-      </lidar>
-      <always_on>1</always_on>
-      <visualize>true</visualize>
-    </sensor>
-  </gazebo>
-    <gazebo>
-        <plugin filename="gz-sim-joint-state-publisher-system" name="gz::sim::systems::JointStatePublisher">
-            <topic>joint_states</topic>
-            <joint_name>right_wheel_joint</joint_name>
-            <joint_name>left_wheel_joint</joint_name>
-        </plugin>
-    </gazebo>
 </robot>
